Commit message: add arm gazebo

File: ur5_description/urdf/ur5.xacro (robot description, xacro)
@@ -1,5 +1,19 @@
 <?xml version="1.0" ?>
 <robot xmlns:xacro="http://www.ros.org/wiki/xacro" name="ur5">
+<xacro:arg name="controller" default="position_control"/>
+<xacro:property name="controller" value="$(arg controller)"/>
+<xacro:if value="${controller == 'position_control'}">
+  <xacro:include filename="$(find ur5_description)/urdf/position_control.gazebo"/>
+</xacro:if>
+<xacro:if value="${controller == 'velocity_control'}">
+  <xacro:include filename="$(find ur5_description)/urdf/velocity_control.gazebo"/>
+</xacro:if>
   <!-- links: main serial chain -->
+  <link name="world"/>
+<joint name="world_to_base" type="fixed">
+  <parent link="world"/>
+  <child link="base_link"/>
+  <origin xyz="0 0 0" rpy="0 0 0"/>
+</joint>
   <link name="base_link"/>
   <link name="base_link_inertia">
@@ -9,7 +23,4 @@
         <mesh filename="file://$(find ur5_description)/meshes/ur5e/visual/base.dae"/>
       </geometry>
-      <material name="LightGrey">
-        <color rgba="0.7 0.7 0.7 1.0"/>
-      </material>
     </visual>
     <collision>
@@ -31,7 +42,4 @@
         <mesh filename="file://$(find ur5_description)/meshes/ur5e/visual/shoulder.dae"/>
       </geometry>
-      <material name="LightGrey">
-        <color rgba="0.7 0.7 0.7 1.0"/>
-      </material>
     </visual>
     <collision>
@@ -53,7 +61,4 @@
         <mesh filename="file://$(find ur5_description)/meshes/ur5e/visual/upperarm.dae"/>
       </geometry>
-      <material name="LightGrey">
-        <color rgba="0.7 0.7 0.7 1.0"/>
-      </material>
     </visual>
     <collision>
@@ -75,7 +80,4 @@
         <mesh filename="file://$(find ur5_description)/meshes/ur5e/visual/forearm.dae"/>
       </geometry>
-      <material name="LightGrey">
-        <color rgba="0.7 0.7 0.7 1.0"/>
-      </material>
     </visual>
     <collision>
@@ -98,7 +100,4 @@
         <mesh filename="file://$(find ur5_description)/meshes/ur5e/visual/wrist1.dae"/>
       </geometry>
-      <material name="LightGrey">
-        <color rgba="0.7 0.7 0.7 1.0"/>
-      </material>
     </visual>
     <collision>
@@ -120,7 +119,4 @@
         <mesh filename="file://$(find ur5_description)/meshes/ur5e/visual/wrist2.dae"/>
       </geometry>
-      <material name="LightGrey">
-        <color rgba="0.7 0.7 0.7 1.0"/>
-      </material>
     </visual>
     <collision>
@@ -142,7 +138,4 @@
         <mesh filename="file://$(find ur5_description)/meshes/ur5e/visual/wrist3.dae"/>
       </geometry>
-      <material name="LightGrey">
-        <color rgba="0.7 0.7 0.7 1.0"/>
-      </material>
     </visual>
     <collision>
@@ -162,9 +155,4 @@
     <parent link="base_link"/>
     <child link="base_link_inertia"/>
-    <!-- 'base_link' is REP-103 aligned (so X+ forward), while the internal
-           frames of the robot/controller have X+ pointing backwards.
-           Use the joint between 'base_link' and 'base_link_inertia' (a dummy
-           link/frame) to introduce the necessary rotation over Z (of pi rad).
-      -->
     <origin rpy="0 0 3.141592653589793" xyz="0 0 0"/>
   </joint>
